Commit message: add collision tags

File: description/robot_core.xacro (robot description, xacro)
@@ -30,4 +30,10 @@
             <material name="white"/>
         </visual>
+        <collision>
+            <origin xyz="0.0 0.0 0.075"/>
+            <geometry>
+                <box size="0.4 0.3 0.15"/>
+            </geometry>
+        </collision>
     </link>
 <!--left front wheel-->
@@ -45,4 +51,9 @@
         <material name="blue"/>
     </visual>
+    <collision>
+        <geometry>
+            <cylinder radius="0.075" length="0.04"/>
+        </geometry>
+    </collision>
 </link>
 <!--right front wheel-->
@@ -60,4 +71,9 @@
         <material name="blue"/>
     </visual>
+    <collision>
+        <geometry>
+            <cylinder radius="0.075" length="0.04"/>
+        </geometry>
+    </collision>
 </link>
 <!--left back wheel-->
@@ -75,4 +91,9 @@
         <material name="blue"/>
     </visual>
+    <collision>
+        <geometry>
+            <cylinder radius="0.075" length="0.04"/>
+        </geometry>
+    </collision>
 </link>
 <!--right back wheel-->
@@ -90,4 +111,9 @@
         <material name="blue"/>
     </visual>
+    <collision>
+        <geometry>
+            <cylinder radius="0.075" length="0.04"/>
+        </geometry>
+    </collision>
 </link>
 </robot>

Commit message: added inertia

File: description/robot_core.xacro (robot description, xacro)
@@ -1,4 +1,5 @@
 <?xml version="1.0"?>
 <robot xmlns:xacro="http://www.ros.org/wiki/xacro" >
+    <xacro:include filename="inertial_macros.xacro"/>
     <material name="white">
         <color rgba="1.0 1.0 1.0 1.0"/>
@@ -36,4 +37,7 @@
             </geometry>
         </collision>
+        <xacro:inertial_box mass="0.5" x="0.3" y="0.3" z="0.15">
+            <origin xyz="0.15 0.0 0.075" rpy="0 0 0"/>
+        </xacro:inertial_box>
     </link>
 <!--left front wheel-->
@@ -56,4 +60,7 @@
         </geometry>
     </collision>
+    <xacro:inertial_cylinder mass="0.1" length="0.04" radius="0.05">
+        <origin xyz="0.0 0.0 0.0" rpy="0.0 0.0 0.0"/>
+    </xacro:inertial_cylinder>
 </link>
 <!--right front wheel-->
@@ -76,4 +83,7 @@
         </geometry>
     </collision>
+    <xacro:inertial_cylinder mass="0.1" length="0.04" radius="0.05">
+        <origin xyz="0.0 0.0 0.0" rpy="0.0 0.0 0.0"/>
+    </xacro:inertial_cylinder>
 </link>
 <!--left back wheel-->
@@ -96,4 +106,7 @@
         </geometry>
     </collision>
+    <xacro:inertial_cylinder mass="0.1" length="0.04" radius="0.05">
+        <origin xyz="0.0 0.0 0.0" rpy="0.0 0.0 0.0"/>
+    </xacro:inertial_cylinder>
 </link>
 <!--right back wheel-->
@@ -116,4 +129,7 @@
         </geometry>
     </collision>
+    <xacro:inertial_cylinder mass="0.1" length="0.04" radius="0.05">
+        <origin xyz="0.0 0.0 0.0" rpy="0.0 0.0 0.0"/>
+    </xacro:inertial_cylinder>
 </link>
 </robot>
