Commit message: new file:   .vscode/settings.json 	new file:   config/my_controllers.yaml 	new file:   description/camera.xacro 	modified:   description/lidar.xacro 	modified:   description/robot.urdf.xacro 	new file:   description/ros2_control.xacro 	new file:   launch/launch_sim_world.launch.py 	new file:   worlds/my_world.world

File: description/lidar.xacro (robot description, xacro)
@@ -4,5 +4,5 @@
         <parent link="chassis"/>
         <child link="laser_frame"/>
-        <origin xyz="0.1 0.0 0.275" rpy="0.0 0.0 0.0"/>
+        <origin xyz="0.1 0.0 0.175" rpy="0.0 0.0 0.0"/>
     </joint>
     <link name="laser_frame">
@@ -32,6 +32,6 @@
                         <samples>360</samples>
                         <resolution>1</resolution>
-                        <min_angles>-3.14</min_angles>
-                        <max_angles>-3.14</max_angles>
+                        <min_angle>-3.14</min_angle>
+                        <max_angle>3.14</max_angle>
                     </horizontal>
                 </scan>

File: description/robot.urdf.xacro (robot description, xacro)
@@ -2,5 +2,7 @@
 <robot xmlns:xacro="http://www.ros.org/wiki/xacro"  name="robot">
     <xacro:include filename="robot_core.xacro"/>
-    <xacro:include  filename="gazebo_control.xacro"/>
+    <!-- <xacro:include filename="gazebo_control.xacro"/> -->
+    <xacro:include filename="ros2_control.xacro"/>
     <xacro:include filename="lidar.xacro"/>
+    <xacro:include filename="camera.xacro"/>
 </robot>
